File: lab4/Exercise1/Exercise1.kicad_sch (KiCad schematic)
At the start: 6 parts, among them J1 Conn_01x02_Male, SW1 SW_SPDT

Commit message: Lab6
Parts:
- 2.2k1: renamed from 2.2k; footprint (none) -> Resistor_THT:R_Axial_DIN0516_L15.5mm_D5.0mm_P20.32mm_Horizontal
- 20K1: renamed from 20K; footprint (none) -> Resistor_THT:R_Axial_DIN0516_L15.5mm_D5.0mm_P20.32mm_Horizontal
- 4.7u1: renamed from 4.7u; footprint (none) -> Capacitor_THT:C_Radial_D5.0mm_H5.0mm_P2.00mm
- D1: footprint (none) -> LED_THT:LED_D5.0mm
- J1: footprint (none) -> Connector_JST:JST_PH_B2B-PH-K_1x02_P2.00mm_Vertical
- SW1: footprint (none) -> Button_Switch_THT:SW_E-Switch_EG1224_SPDT_Angled
Changed lines of the file:
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@@
       (effects (font (size 1.27 1.27)) (justify right))
     )
-    (property "Footprint" "" (id 2) (at 171.45 74.93 0)
+    (property "Footprint" "LED_THT:LED_D5.0mm" (id 2) (at 171.45 74.93 0)
       (effects (font (size 1.27 1.27)) hide)
     )
@@
   (symbol (lib_id "Device:R") (at 158.75 71.12 90) (unit 1)
     (in_bom yes) (on_board yes) (fields_autoplaced)
-    (property "Reference" "20K" (id 0) (at 158.75 64.77 90))
+    (property "Reference" "20K1" (id 0) (at 158.75 64.77 90))
     (property "Value" "R1" (id 1) (at 158.75 67.31 90))
-    (property "Footprint" "" (id 2) (at 158.75 72.898 90)
+    (property "Footprint" "Resistor_THT:R_Axial_DIN0516_L15.5mm_D5.0mm_P20.32mm_Horizontal" (id 2) (at 158.75 72.898 90)
       (effects (font (size 1.27 1.27)) hide)
     )
@@
   (symbol (lib_id "Device:R") (at 123.19 71.12 90) (unit 1)
     (in_bom yes) (on_board yes) (fields_autoplaced)
-    (property "Reference" "2.2k" (id 0) (at 123.19 64.77 90))
+    (property "Reference" "2.2k1" (id 0) (at 123.19 64.77 90))
     (property "Value" "R2" (id 1) (at 123.19 67.31 90))
-    (property "Footprint" "" (id 2) (at 123.19 72.898 90)
+    (property "Footprint" "Resistor_THT:R_Axial_DIN0516_L15.5mm_D5.0mm_P20.32mm_Horizontal" (id 2) (at 123.19 72.898 90)
       (effects (font (size 1.27 1.27)) hide)
     )
@@
   (symbol (lib_id "Device:C_Polarized") (at 146.05 74.93 0) (unit 1)
     (in_bom yes) (on_board yes) (fields_autoplaced)
-    (property "Reference" "4.7u" (id 0) (at 149.86 72.7709 0)
+    (property "Reference" "4.7u1" (id 0) (at 149.86 72.7709 0)
       (effects (font (size 1.27 1.27)) (justify left))
     )
@@
       (effects (font (size 1.27 1.27)) (justify left))
     )
-    (property "Footprint" "" (id 2) (at 147.0152 78.74 0)
+    (property "Footprint" "Capacitor_THT:C_Radial_D5.0mm_H5.0mm_P2.00mm" (id 2) (at 147.0152 78.74 0)
       (effects (font (size 1.27 1.27)) hide)
     )
@@
     (property "Reference" "J1" (id 0) (at 109.855 66.04 0))
     (property "Value" "Conn_01x02_Male" (id 1) (at 109.855 68.58 0))
-    (property "Footprint" "" (id 2) (at 109.22 71.12 0)
+    (property "Footprint" "Connector_JST:JST_PH_B2B-PH-K_1x02_P2.00mm_Vertical" (id 2) (at 109.22 71.12 0)
       (effects (font (size 1.27 1.27)) hide)
     )
@@
     (property "Reference" "SW1" (id 0) (at 135.89 60.96 0))
     (property "Value" "SW_SPDT" (id 1) (at 135.89 63.5 0))
-    (property "Footprint" "" (id 2) (at 135.89 68.58 0)
+    (property "Footprint" "Button_Switch_THT:SW_E-Switch_EG1224_SPDT_Angled" (id 2) (at 135.89 68.58 0)
       (effects (font (size 1.27 1.27)) hide)
     )
@@
   (symbol_instances
     (path "/34f3d410-2523-4f8b-95ad-e2400a90ebc4"
-      (reference "2.2k") (unit 1) (value "R2") (footprint "")
+      (reference "2.2k1") (unit 1) (value "R2") (footprint "Resistor_THT:R_Axial_DIN0516_L15.5mm_D5.0mm_P20.32mm_Horizontal")
     )
     (path "/7fcffb4b-894b-48f4-9e38-759303b9263c"
-      (reference "4.7u") (unit 1) (value "C_Polarized") (footprint "")
+      (reference "4.7u1") (unit 1) (value "C_Polarized") (footprint "Capacitor_THT:C_Radial_D5.0mm_H5.0mm_P2.00mm")
     )
     (path "/1e018703-0583-433b-8f9d-4f6a19aab353"
-      (reference "20K") (unit 1) (value "R1") (footprint "")
+      (reference "20K1") (unit 1) (value "R1") (footprint "Resistor_THT:R_Axial_DIN0516_L15.5mm_D5.0mm_P20.32mm_Horizontal")
     )
     (path "/008f58c4-0506-4a84-8b5d-82ba4713cb7a"
-      (reference "D1") (unit 1) (value "LED") (footprint "")
+      (reference "D1") (unit 1) (value "LED") (footprint "LED_THT:LED_D5.0mm")
     )
     (path "/b04c841f-f5c8-4768-a837-c6c49d965337"
-      (reference "J1") (unit 1) (value "Conn_01x02_Male") (footprint "")
+      (reference "J1") (unit 1) (value "Conn_01x02_Male") (footprint "Connector_JST:JST_PH_B2B-PH-K_1x02_P2.00mm_Vertical")
     )
     (path "/fd634884-0b55-4e2a-8a3e-5abb1750244b"
-      (reference "SW1") (unit 1) (value "SW_SPDT") (footprint "")
+      (reference "SW1") (unit 1) (value "SW_SPDT") (footprint "Button_Switch_THT:SW_E-Switch_EG1224_SPDT_Angled")
     )
   )
